File: MFOS Dual VCA Sliders.brd (EAGLE design)
At the start: 97.5 x 49.5 mm, 61 parts, among them IC1 TL072P, IC2 LM13700N, Q1 2N3904, Q2 2N3904, Q3 2N3906, Q4 2N3906, U1 POWER

Commit message: url on board
Parts:
- moved R15 14.0 mm to (48.3, 40.0)
- moved R21 2.84 mm to (20.3, 33.7), flipped to the top, turned to 0 degrees
- moved Q2 2.01 mm to (55.2, 22.9), turned to 0 degrees
- moved Q3 1.27 mm to (14.0, 31.1)
- moved R28 1.27 mm to (5.08, 22.2), turned to 180 degrees
- moved R18 0.63 mm to (29.2, 21.0)
- turned C21 to 270 degrees
- turned C24 to 90 degrees
Routing:
- net N$30: track 115.8 -> 177.8 mm, vias 1 -> 0
- net N$15: track 36.3 -> 15.9 mm
- net GND: track 328.8 -> 310.2 mm, vias 3 -> 2
- net N$6: track 40.8 -> 55.4 mm
- net +12V: track 238.8 -> 252.5 mm
- net N$20: track 103.1 -> 94.4 mm, vias 1 -> 3
- net -12V: track 200.6 -> 208.8 mm, vias 2 -> 4
- net N$23: track 90.8 -> 85.3 mm
- net N$9: track 56.3 -> 61.7 mm, vias 0 -> 1
- net N$14: track 55.5 -> 51.9 mm, vias 2 -> 1
- net N$7: track 54.2 -> 50.9 mm, vias 2 -> 1
- net N$29: track 8.83 -> 5.48 mm
- net N$8: track 10.1 -> 8.98 mm
- net N$12: track 6.17 -> 6.86 mm
- net N$21: track 25.3 -> 25.8 mm
Other:
- board text added: "Release v0.1"
- board text added: "https://github.com/jbeuckm/MFOS-Dual-VCA-Sliders"
